Commit message: Start new repository with old rastreator code

File: rastreator/rastreator_description/urdf/rastreator.urdf (robot description, URDF)
Before this commit: robot rastreator, 9 links, 8 joints
Links:
- removed link d435_link
- removed link lidar_link
- removed link t265_link
- added link sensor_laser, mass 0.1; collision mesh filename=package://rastreator_description/mesh/rplidar_a3.stl scale=0.001 0.001 0.001; visual mesh filename=package://rastreator_description/mesh/rplidar_a3.stl scale=0.001 0.001 0.001
- link base_link: mass 2.0 -> 1.0
- link imu_link: mass 0.01 -> None
- link left_wheel_link: mass 0.3 -> 0.15
- link right_wheel_link: mass 0.3 -> 0.15
Joints:
- removed joint d435_joint
- removed joint lidar_joint
- removed joint t265_joint
- added joint sensor_laser_joint: type fixed, parent base_link, child sensor_laser, origin xyz=0.0 0.0 0.132 rpy=0 0.0 0
- joint base_joint: origin xyz=0.0 0.0 0.0205 rpy=0 0 0 -> xyz=0.0 0.0 0.0235 rpy=0 0 0
- joint wheel_left_joint: origin xyz=-0.042 0.078 0.012 rpy=0 0 0 -> xyz=-0.075 0.076 0.01501 rpy=0 0 0
- joint wheel_right_joint: origin xyz=-0.045 -0.08 0.012 rpy=0 0 0 -> xyz=-0.075 -0.081 0.01501 rpy=0 0 0

File: rastreator/rastreator_description/urdf/rastreator.xacro (robot description, xacro)
@@ -5,5 +5,5 @@
     <!--**************************************************************-->
     <!--base_link-->
-    <xacro:property name="base_mass" value="2.0"/>
+    <xacro:property name="base_mass" value="1.0"/>
     <xacro:property name="base_width" value="0.142"/>
     <xacro:property name="base_len" value="0.2"/>
@@ -11,28 +11,16 @@
     <xacro:property name="plate_height" value="0.00849"/>
     <!--wheels-->
-    <xacro:property name="wheel_mass" value="0.3"/>
+    <xacro:property name="wheel_mass" value="0.15"/>
     <xacro:property name="wheel_radius" value="0.0325"/>
+    <xacro:property name="wheel_diameter" value="0.065"/>
+    <xacro:property name="wheel_separation" value="0.16"/>
     <xacro:property name="wheel_height" value="0.018"/>
-    <xacro:property name="wheel_separation" value="0.16"/>
+    <xacro:property name="wheel_x_pos" value="0.075"/>
+    <xacro:property name="wheel_left_offset" value="0.004"/>
+    <xacro:property name="wheel_right_offset" value="0.001"/>
+    <!--front caster wheel-->
+    <xacro:property name="caster_height" value="0.009"/>
     <xacro:property name="wheel_torque" value="10"/>
     <xacro:property name="wheel_acc" value="1.0"/>
-    <!--right wheel position-->
-    <xacro:property name="wheel_right_x" value="-0.045"/>
-    <xacro:property name="wheel_right_y" value="-0.080"/>
-    <xacro:property name="wheel_right_z" value="0.012"/>
-    <!--left wheel  position-->
-    <xacro:property name="wheel_left_x" value="-0.042"/>
-    <xacro:property name="wheel_left_y" value="0.078"/>
-    <xacro:property name="wheel_left_z" value="0.012"/>
-    <!--front caster wheel position-->
-    <xacro:property name="caster_height" value="0.012"/>
-    <!--camera D435  position-->
-    <xacro:property name="camera_d435_x" value="0.117"/>
-    <xacro:property name="camera_d435_y" value="-0.014"/>
-    <xacro:property name="camera_d435_z" value="0.112"/>
-    <!--camera T265  position-->
-    <xacro:property name="camera_t265_x" value="0.117"/>
-    <xacro:property name="camera_t265_y" value="-0.005"/>
-    <xacro:property name="camera_t265_z" value="0.087"/>
     <xacro:property name="update_rate" value="30"/>
     <!--**************************************************************-->
@@ -124,5 +112,5 @@
     <!--JOINT-->
     <joint name='wheel_left_joint' type='continuous'>
-      <origin xyz="${wheel_left_x} ${wheel_left_y} ${wheel_left_z}" rpy="0 0 0"/>
+      <origin xyz="-${wheel_x_pos} ${(wheel_separation/2)-wheel_left_offset} ${wheel_radius-caster_height-plate_height}" rpy="0 0 0"/>
       <child  link="left_wheel_link"/>
       <parent link="base_link"/>
@@ -151,5 +139,5 @@
     <!--JOINT-->
     <joint name='wheel_right_joint' type='continuous'>
-      <origin xyz="${wheel_right_x} ${wheel_right_y} ${wheel_right_z}" rpy="0 0 0"/>
+      <origin xyz="-${wheel_x_pos} -${(wheel_separation/2)+wheel_right_offset} ${wheel_radius-caster_height-plate_height}" rpy="0 0 0"/>
       <child  link="right_wheel_link"/>
       <parent link="base_link"/>
@@ -189,9 +177,11 @@
     <!--LASER/LIDAR-->
     <!--**************************************************************-->
-    <link name="lidar_link">
-      <inertial>
-        <inertia ixx="0.0" ixy="0.0" ixz="0.0" iyy="0.0" iyz="0.0" izz="0.0"/>
+    <link name="sensor_laser">
+      <!--INERTIA-->
+      <inertial>
+        <inertia ixx="0"  ixy="0"  ixz="0" iyy="0" iyz="0" izz="0" />
         <mass value="0.1"/>
       </inertial>
+      <!--COLLISION-->
       <collision>
         <geometry>
@@ -199,4 +189,6 @@
         </geometry>
       </collision>
+      <gravity>false</gravity>
+      <!--VISUAL-->
       <visual>
         <geometry>
@@ -206,72 +198,14 @@
       </visual>
     </link>
-    <joint name="lidar_joint" type="fixed">
-        <origin rpy="0 0.0 0" xyz="0.0 0.0 ${base_height}"/>
-        <child  link="lidar_link"/>
+    <!--JOINT-->
+    <joint name="sensor_laser_joint" type="fixed">
+        <origin rpy="0 0.0 0" xyz="0.0 0.0 ${base_height+0.005}"/>
+        <child  link="sensor_laser"/>
         <parent link="base_link"/>
     </joint>
     <!--**************************************************************-->
-    <!--CAMERA T265-->
-    <!--**************************************************************-->
-    <link name="t265_link">
-      <!--INERTIA-->
-      <!--Not calling macro, just small values-->
-      <inertial>
-        <mass value="0.005"/>
-        <inertia ixx="0.001" ixy="0.0" ixz="0.0" iyy="0.001" iyz="0.0" izz="0.001"/>
-      </inertial>
-      <collision>
-        <geometry>
-          <mesh filename="package://rastreator_description/mesh/intelrealsenseT265.stl" scale="0.001 0.001 0.001"/>
-        </geometry>
-      </collision>
-      <visual>
-        <geometry>
-          <mesh filename="package://rastreator_description/mesh/intelrealsenseT265.stl" scale="0.001 0.001 0.001"/>
-        </geometry>
-        <material name="dark"/>
-      </visual>
-    </link>
-    <joint name="t265_joint" type="fixed">
-      <origin rpy="0 0 0" xyz="${camera_t265_x} ${camera_t265_y} ${camera_t265_z}"/>
-      <child  link="t265_link"/>
-      <parent link="base_link"/>
-    </joint>
-    <!--**************************************************************-->
-    <!--CAMERA D435-->
-    <!--**************************************************************-->
-    <link name="d435_link">
-      <!--INERTIA-->
-      <!--Not calling macro, just small values-->
-      <inertial>
-        <mass value="0.005"/>
-        <inertia ixx="0.001" ixy="0.0" ixz="0.0" iyy="0.001" iyz="0.0" izz="0.001"/>
-      </inertial>
-      <collision>
-        <geometry>
-          <mesh filename="package://rastreator_description/mesh/intelrealsenseD435.stl" scale="0.001 0.001 0.001"/>
-        </geometry>
-      </collision>
-      <visual>
-        <geometry>
-          <mesh filename="package://rastreator_description/mesh/intelrealsenseD435.stl" scale="0.001 0.001 0.001"/>
-        </geometry>
-        <material name="dark"/>
-      </visual>
-    </link>
-    <joint name="d435_joint" type="fixed">
-      <origin rpy="0 0 0" xyz="${camera_d435_x} ${camera_d435_y} ${camera_d435_z}"/>
-      <child  link="d435_link"/>
-      <parent link="base_link"/>
-    </joint>
-    <!--**************************************************************-->
     <!--IMU-->
     <!--**************************************************************-->
     <link name="imu_link">
-      <!--INERTIA-->
-        <inertial>
-          <inertia ixx="0.001" ixy="0.0" ixz="0.0" iyy="0.001" iyz="0.0" izz="0.001"/>
-          <mass value="0.01"/>
-        </inertial>
         <!--COLLISION-->
         <collision>
@@ -288,4 +222,16 @@
           <material name="dark"/>
         </visual>
+        <!--
+        <sensor name="rastreator_imu" type="imu">
+          <always_on>true</always_on>
+          <update_rate>${update_rate}</update_rate>
+          <plugin name="imu" filename="libgazebo_ros_imu_sensor.so">
+            <ros>
+              <namespace>/sim</namespace>
+              <argument>~/out:=imu_sim</argument>
+            </ros>
+          </plugin>
+        </sensor>
+        -->
     </link>
     <!--JOINT-->
@@ -300,7 +246,4 @@
     <gazebo reference="base_link">
       <material>Gazebo/DarkGrey</material>
-    </gazebo>
-    <gazebo reference="imu_link">
-      <material>Gazebo/FlatBlack</material>
     </gazebo>
     <gazebo reference="left_wheel_link">
@@ -329,12 +272,12 @@
       <mu2>0.1</mu2>
       <kp>1000000.0</kp>
-      <kd>10.0</kd>
+      <kd>100.0</kd>
       <minDepth>0.001</minDepth>
       <maxVel>1.0</maxVel>
     </gazebo>
-    <gazebo reference="t265_link">
-      <material>Gazebo/FlatBlack</material>
-    </gazebo>
-    <gazebo reference="d435_link">
+    <gazebo reference="sensor_laser">
+      <material>Gazebo/FlatBlack</material>
+    </gazebo>
+    <gazebo reference="imu_link">
       <material>Gazebo/FlatBlack</material>
     </gazebo>
@@ -363,5 +306,5 @@
       <right_joint>wheel_right_joint</right_joint>
       <wheel_separation>${wheel_separation}</wheel_separation>
-      <wheel_diameter>${wheel_radius*2}</wheel_diameter>
+      <wheel_diameter>${wheel_diameter}</wheel_diameter>
       <max_wheel_torque>${wheel_torque}</max_wheel_torque>
       <max_wheel_acceleration>${wheel_acc}</max_wheel_acceleration>
@@ -389,67 +332,4 @@
         <gaussian_noise>0</gaussian_noise>
       </plugin>
-  </gazebo>
-  <!--lidar-->
-  <gazebo reference="lidar_link">
-      <material>Gazebo/FlatBlack</material>
-      <inertial>
-        <inertia>
-          <ixx>0.001</ixx>
-          <ixy>0.000</ixy>
-          <ixz>0.000</ixz>
-          <iyy>0.001</iyy>
-          <iyz>0.000</iyz>
-          <izz>0.001</izz>
-        </inertia>
-        <mass>0.125</mass>
-      </inertial>
-      <collision name="lidar_link_sensor_collision">
-        <geometry>
-          <cylinder>
-            <radius>0.0508</radius>
-            <length>0.055</length>
-          </cylinder>
-        </geometry>
-      </collision>
-      <visual name="lidar_link_sensor_visual">
-        <geometry>
-          <mesh>
-            <uri>model://rastreator_description/mesh/rplidar_a3.stl</uri>
-            <scale>0.001 0.001 0.001</scale>
-          </mesh>
-        </geometry>
-      </visual>
-      <sensor name="lidar_plugin" type="ray">
-        <always_on>true</always_on>
-        <visualize>true</visualize>
-        <update_rate>${update_rate}</update_rate>
-        <ray>
-          <scan>
-            <horizontal>
-              <samples>360</samples>
-              <resolution>1.000000</resolution>
-              <min_angle>0.000000</min_angle>
-              <max_angle>6.280000</max_angle>
-            </horizontal>
-          </scan>
-          <range>
-            <min>0.120000</min>
-            <max>3.5</max>
-            <resolution>0.015000</resolution>
-          </range>
-          <noise>
-            <type>gaussian</type>
-            <mean>0.0</mean>
-            <stddev>0.01</stddev>
-          </noise>
-        </ray>
-        <plugin name="plugin_lidar" filename="libgazebo_ros_ray_sensor.so">
-          <ros>
-            <argument>~/out:=scan</argument>
-          </ros>
-          <output_type>sensor_msgs/LaserScan</output_type>
-          <frame_name>lidar_link</frame_name>
-        </plugin>
-      </sensor>
-  </gazebo>
+    </gazebo>
 </robot>

Commit message: rastreator bringup add camera and description urdf

File: rastreator/rastreator_description/urdf/rastreator.urdf (robot description, URDF)
Before this commit: robot rastreator, 9 links, 8 joints
Links:
- removed link d435_link
- added link camera, mass 0.005; collision mesh filename=package://rastreator_description/mesh/intelrealsenseD435.stl scale=0.001 0.001 0.001; visual mesh filename=package://rastreator_description/mesh/intelrealsenseD435.stl scale=0.001 0.001 0.001
Joints:
- removed joint d435_joint
- added joint camera_joint: type fixed, parent base_link, child camera, origin xyz=0.117 -0.014 0.112 rpy=0 0 0

File: rastreator/rastreator_description/urdf/rastreator.xacro (robot description, xacro)
@@ -239,7 +239,7 @@
     </joint>
     <!--**************************************************************-->
-    <!--CAMERA D435-->
-    <!--**************************************************************-->
-    <link name="d435_link">
+    <!--CAMERA D435 | CSI CAM, testing (change d435 for camera) -->
+    <!--**************************************************************-->
+    <link name="camera">
       <!--INERTIA-->
       <!--Not calling macro, just small values-->
@@ -260,7 +260,7 @@
       </visual>
     </link>
-    <joint name="d435_joint" type="fixed">
+    <joint name="camera_joint" type="fixed">
       <origin rpy="0 0 0" xyz="${camera_d435_x} ${camera_d435_y} ${camera_d435_z}"/>
-      <child  link="d435_link"/>
+      <child  link="camera"/>
       <parent link="base_link"/>
     </joint>
@@ -336,5 +336,5 @@
       <material>Gazebo/FlatBlack</material>
     </gazebo>
-    <gazebo reference="d435_link">
+    <gazebo reference="camera_link">
       <material>Gazebo/FlatBlack</material>
     </gazebo>
@@ -421,6 +421,6 @@
       </visual>
       <sensor name="lidar_plugin" type="ray">
-        <always_on>true</always_on>
-        <visualize>true</visualize>
+        <always_on>false</always_on>
+        <visualize>false</visualize>
         <update_rate>${update_rate}</update_rate>
         <ray>
