Commit message: testing ORB

File: rastreator/rastreator_description/urdf/rastreator_intelrealsense.urdf (robot description, URDF)
Before this commit: robot rastreator, 9 links, 8 joints
Links:
- removed link camera
- added link d435_link, mass 0.005; collision mesh filename=package://rastreator_description/mesh/intelrealsenseD435.stl scale=0.001 0.001 0.001; visual mesh filename=package://rastreator_description/mesh/intelrealsenseD435.stl scale=0.001 0.001 0.001
Joints:
- joint camera_joint: child camera -> d435_link

File: rastreator/rastreator_description/urdf/rastreator_intelrealsense.xacro (robot description, xacro)
@@ -239,7 +239,7 @@
     </joint>
     <!--**************************************************************-->
-    <!--CAMERA D435 | CSI CAM, testing (change d435 for camera) -->
-    <!--**************************************************************-->
-    <link name="camera">
+    <!--CAMERA D435-->
+    <!--**************************************************************-->
+    <link name="d435_link">
       <!--INERTIA-->
       <!--Not calling macro, just small values-->
@@ -262,5 +262,5 @@
     <joint name="camera_joint" type="fixed">
       <origin rpy="0 0 0" xyz="${camera_d435_x} ${camera_d435_y} ${camera_d435_z}"/>
-      <child  link="camera"/>
+      <child  link="d435_link"/>
       <parent link="base_link"/>
     </joint>
@@ -336,5 +336,5 @@
       <material>Gazebo/FlatBlack</material>
     </gazebo>
-    <gazebo reference="camera_link">
+    <gazebo reference="d435_link">
       <material>Gazebo/FlatBlack</material>
     </gazebo>
