Commit message: orb testing

File: rastreator/rastreator_description/urdf/rastreator_csicam.urdf (robot description, URDF)
Before this commit: robot rastreator, 8 links, 7 joints
Links:
- removed link odom
- added link base_footprint
Joints:
- joint base_joint: parent odom -> base_footprint
- joint camera_joint: parent odom -> base_link

File: rastreator/rastreator_description/urdf/rastreator_csicam.xacro (robot description, xacro)
@@ -69,7 +69,7 @@
     </xacro:macro>
     <!--**************************************************************-->
-    <!--ODOM-->
-    <!--**************************************************************-->
-    <link name="odom"/>
+    <!--DUUMY LINK-->
+    <!--**************************************************************-->
+    <link name="base_footprint"/>
     <!--**************************************************************-->
     <!--CHASSIS (base link)-->
@@ -95,5 +95,5 @@
     <joint name="base_joint" type="fixed">
       <origin xyz="0.0 0.0 ${wheel_radius-caster_height}" rpy="0 0 0"/>
-      <parent link="odom"/>
+      <parent link="base_footprint"/>
       <child link="base_link" />
     </joint>
@@ -214,5 +214,5 @@
       <origin rpy="0 0 0" xyz="${camera_d435_x} ${camera_d435_y} ${camera_d435_z}"/>
       <child  link="csicam_link"/>
-      <parent link="odom"/>
+      <parent link="base_link"/>
     </joint>
     <!--**************************************************************-->
